File: KiCAD Files/Vertigo Flight Computers/Vertigo Pro/Vertigo Pro PR1/Vertigo Pro PR1.kicad_sch (KiCad schematic)
At the start: 138 parts, among them IC1 ICM-20602, IC2 DPS310XTSA1, J1 ST-LINK Conn, J2 USB_C_2.0, J3 FFC2A32-24-T, J4 Screw_Terminal, J5 Screw_Terminal, J6 Screw_Terminal, J7 Screw_Terminal, Q1 IRF530SPBF, Q2 MMBT3904-TP, Q3 MMBT3904-TP, Q4 IRF530SPBF, Q5 SI7149ADP-T1-GE3, Q6 MMBT3904-TP, Q7 MMBT3904-TP, Q8 IRF530SPBF, Q9 IRF530SPBF, SW1 SW_SPDT, U1 STM32F103C8Tx, U10 TPS79133DBVR, U11 TLV709, U12 TLV709, U13 TLV75528PDBV, U2 AP63203WU, U3 ESP32-S3-WROOM-1, U4 TLV75515PDBV, U8 NEO-6M-GPS, U9 24AA32A-I_MS, Y1 16MHz

Commit message: fix
Other:
- note added: "Protects VBUS from ESD"
- note removed: "uClamp0571 Protects VBUS from ESD"
Changed lines of the file:
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@@
 	)
 	(junction
+		(at 403.86 199.39)
+		(diameter 0)
+		(color 0 0 0 0)
+	)
+	(junction
 		(at 213.36 163.83)
 		(diameter 0)
@@
 	)
 	(junction
-		(at 402.59 199.39)
-		(diameter 0)
-		(color 0 0 0 0)
-	)
-	(junction
 		(at 223.52 163.83)
 		(diameter 0)
@@
 	(wire
 		(pts
-			(xy 480.06 167.64) (xy 485.14 167.64)
-		)
-		(stroke
-			(width 0)
-			(type default)
-		)
-	)
-	(wire
-		(pts
 			(xy 403.86 227.33) (xy 403.86 226.06)
 		)
@@
 	(wire
 		(pts
-			(xy 556.26 163.83) (xy 565.15 163.83)
+			(xy 146.05 316.23) (xy 146.05 320.04)
 		)
 		(stroke
@@
 	(wire
 		(pts
-			(xy 58.42 262.89) (xy 58.42 261.62)
+			(xy 556.26 163.83) (xy 565.15 163.83)
 		)
 		(stroke
@@
 	(wire
 		(pts
-			(xy 146.05 323.85) (xy 146.05 320.04)
+			(xy 58.42 262.89) (xy 58.42 261.62)
 		)
 		(stroke
@@
 	(wire
 		(pts
-			(xy 146.05 313.69) (xy 152.4 313.69)
+			(xy 149.86 313.69) (xy 152.4 313.69)
 		)
 		(stroke
@@
 	(wire
 		(pts
-			(xy 494.03 288.29) (xy 501.65 288.29)
-		)
-		(stroke
-			(width 0)
-			(type default)
-		)
-	)
-	(wire
-		(pts
 			(xy 116.84 63.5) (xy 116.84 71.12)
 		)
@@
 	(wire
 		(pts
-			(xy 389.89 199.39) (xy 402.59 199.39)
+			(xy 389.89 199.39) (xy 403.86 199.39)
 		)
 		(stroke
@@
 	(wire
 		(pts
-			(xy 494.03 288.29) (xy 494.03 300.99)
+			(xy 501.65 288.29) (xy 501.65 285.75)
 		)
 		(stroke
@@
 	(wire
 		(pts
-			(xy 508 120.65) (xy 518.16 120.65)
-		)
-		(stroke
-			(width 0)
-			(type default)
-		)
-	)
-	(wire
-		(pts
 			(xy 532.13 167.64) (xy 532.13 168.91)
 		)
@@
 	(wire
 		(pts
+			(xy 403.86 199.39) (xy 411.48 199.39)
+		)
+		(stroke
+			(width 0)
+			(type default)
+		)
+	)
+	(wire
+		(pts
 			(xy 69.85 219.71) (xy 69.85 218.44)
 		)
@@
 	(wire
 		(pts
-			(xy 402.59 199.39) (xy 411.48 199.39)
-		)
-		(stroke
-			(width 0)
-			(type default)
-		)
-	)
-	(wire
-		(pts
 			(xy 187.96 168.91) (xy 184.15 168.91)
 		)
@@
 	(wire
 		(pts
-			(xy 402.59 196.85) (xy 402.59 199.39)
+			(xy 403.86 196.85) (xy 403.86 199.39)
 		)
 		(stroke
@@
 	(wire
 		(pts
-			(xy 146.05 313.69) (xy 146.05 314.96)
+			(xy 149.86 313.69) (xy 149.86 314.96)
 		)
 		(stroke
@@
 	(wire
 		(pts
-			(xy 480.06 167.64) (xy 480.06 180.34)
+			(xy 485.14 167.64) (xy 485.14 165.1)
 		)
 		(stroke
@@
 	(wire
 		(pts
-			(xy 508 120.65) (xy 508 132.08)
+			(xy 518.16 120.65) (xy 518.16 118.11)
 		)
 		(stroke
@@
 	(wire
 		(pts
-			(xy 134.62 320.04) (xy 146.05 320.04)
+			(xy 133.35 320.04) (xy 146.05 320.04)
 		)
 		(stroke
@@
 		)
 	)
-	(text "uClamp0571 Protects \nVBUS from ESD"
+	(text "Protects VBUS from ESD"
 		(exclude_from_sim no)
-		(at 176.53 330.2 0)
+		(at 176.53 328.93 0)
 		(effects
 			(font
@@
 	(text "R3,R2=22R"
 		(exclude_from_sim no)
-		(at 129.54 317.5 0)
+		(at 129.54 316.23 0)
 		(effects
 			(font
@@
 	(text "Protection agains diode failure"
 		(exclude_from_sim no)
-		(at 172.72 339.09 0)
+		(at 173.99 337.82 0)
 		(effects
 			(font
@@
 	)
 	(label "5V_USB_RAW"
-		(at 134.62 320.04 0)
+		(at 133.35 320.04 0)
 		(fields_autoplaced yes)
 		(effects
@@
 	(symbol
 		(lib_id "power:GND")
-		(at 146.05 314.96 0)
+		(at 149.86 314.96 0)
 		(unit 1)
 		(exclude_from_sim no)
@@
 		(fields_autoplaced yes)
 		(property "Reference" "#PWR016"
-			(at 146.05 321.31 0)
+			(at 149.86 321.31 0)
 			(effects
 				(font
@@
 		)
 		(property "Value" "GND"
-			(at 146.05 320.04 0)
+			(at 149.86 320.04 0)
 			(effects
 				(font
@@
 		)
 		(property "Footprint" ""
-			(at 146.05 314.96 0)
+			(at 149.86 314.96 0)
 			(effects
 				(font
@@
 		)
 		(property "Datasheet" ""
-			(at 146.05 314.96 0)
+			(at 149.86 314.96 0)
 			(effects
 				(font
@@
 		)
 		(property "Description" ""
-			(at 146.05 314.96 0)
+			(at 149.86 314.96 0)
 			(effects
 				(font
@@
 	(symbol
 		(lib_id "power:VCC")
-		(at 508 132.08 180)
+		(at 518.16 118.11 0)
 		(unit 1)
 		(exclude_from_sim no)
@@
 		(dnp no)
 		(property "Reference" "#PWR058"
-			(at 508 128.27 0)
+			(at 518.16 121.92 0)
 			(effects
 				(font
@@
 		)
 		(property "Value" "VCC"
-			(at 508 135.89 0)
+			(at 518.16 114.3 0)
 			(effects
 				(font
@@
 		)
 		(property "Footprint" ""
-			(at 508 132.08 0)
+			(at 518.16 118.11 0)
 			(effects
 				(font
@@
 		)
 		(property "Datasheet" ""
-			(at 508 132.08 0)
+			(at 518.16 118.11 0)
 			(effects
 				(font
@@
 		)
 		(property "Description" "Power symbol creates a global label with name \"VCC\""
-			(at 508 132.08 0)
+			(at 518.16 118.11 0)
 			(effects
 				(font
@@
 		(dnp no)
 		(property "Reference" "D3"
-			(at 151.13 317.5 0)
+			(at 152.4 317.5 0)
 			(effects
 				(font
@@
 	(symbol
 		(lib_id "power:VCC")
-		(at 494.03 300.99 180)
+		(at 501.65 285.75 0)
 		(unit 1)
 		(exclude_from_sim no)
@@
 		(dnp no)
 		(property "Reference" "#PWR056"
-			(at 494.03 297.18 0)
+			(at 501.65 289.56 0)
 			(effects
 				(font
@@
 		)
 		(property "Value" "VCC"
-			(at 494.03 304.8 0)
+			(at 501.65 281.94 0)
 			(effects
 				(font
@@
 		)
 		(property "Footprint" ""
-			(at 494.03 300.99 0)
+			(at 501.65 285.75 0)
 			(effects
 				(font
@@
 		)
 		(property "Datasheet" ""
-			(at 494.03 300.99 0)
+			(at 501.65 285.75 0)
 			(effects
 				(font
@@
 		)
 		(property "Description" "Power symbol creates a global label with name \"VCC\""
-			(at 494.03 300.99 0)
+			(at 501.65 285.75 0)
 			(effects
 				(font
@@
 	(symbol
 		(lib_id "power:VCC")
-		(at 480.06 180.34 180)
+		(at 485.14 165.1 0)
 		(unit 1)
 		(exclude_from_sim no)
@@
 		(dnp no)
 		(property "Reference" "#PWR057"
-			(at 480.06 176.53 0)
+			(at 485.14 168.91 0)
 			(effects
 				(font
@@
 		)
 		(property "Value" "VCC"
-			(at 480.06 184.15 0)
+			(at 485.14 161.29 0)
 			(effects
 				(font
@@
 		)
 		(property "Footprint" ""
-			(at 480.06 180.34 0)
+			(at 485.14 165.1 0)
 			(effects
 				(font
@@
 		)
 		(property "Datasheet" ""
-			(at 480.06 180.34 0)
+			(at 485.14 165.1 0)
 			(effects
 				(font
@@
 		)
 		(property "Description" "Power symbol creates a global label with name \"VCC\""
-			(at 480.06 180.34 0)
+			(at 485.14 165.1 0)
 			(effects
 				(font
@@
 	(symbol
 		(lib_id "power:VCC")
-		(at 402.59 196.85 0)
+		(at 403.86 196.85 0)
 		(unit 1)
 		(exclude_from_sim no)
@@
 		(dnp no)
 		(property "Reference" "#PWR054"
-			(at 402.59 200.66 0)
+			(at 403.86 200.66 0)
 			(effects
 				(font
@@
 		)
 		(property "Value" "VCC"
-			(at 402.59 193.04 0)
+			(at 403.86 193.04 0)
 			(effects
 				(font
@@
 		)
 		(property "Footprint" ""
-			(at 402.59 196.85 0)
+			(at 403.86 196.85 0)
 			(effects
 				(font
@@
 		)
 		(property "Datasheet" ""
-			(at 402.59 196.85 0)
+			(at 403.86 196.85 0)
 			(effects
 				(font
@@
 		)
 		(property "Description" "Power symbol creates a global label with name \"VCC\""
-			(at 402.59 196.85 0)
+			(at 403.86 196.85 0)
 			(effects
 				(font
@@
 	(symbol
 		(lib_id "power:VCC")
-		(at 146.05 323.85 180)
+		(at 146.05 316.23 0)
 		(unit 1)
 		(exclude_from_sim no)
@@
 		)
 		(property "Value" "VCC"
-			(at 146.05 327.66 0)
+			(at 146.05 312.42 0)
 			(effects
 				(font
@@
 		)
 		(property "Footprint" ""
-			(at 146.05 323.85 0)
+			(at 146.05 316.23 0)
 			(effects
 				(font
@@
 		)
 		(property "Datasheet" ""
-			(at 146.05 323.85 0)
+			(at 146.05 316.23 0)
 			(effects
 				(font
@@
 		)
 		(property "Description" "Power symbol creates a global label with name \"VCC\""
-			(at 146.05 323.85 0)
+			(at 146.05 316.23 0)
 			(effects
 				(font
