File: KiCAD Files/Vertigo Flight Computers/Vertigo Pro/Vertigo Pro PR1/_autosave-Vertigo Pro PR1.kicad_sch (KiCad schematic)
At the start: 132 parts, among them IC1 ICM-20602, IC2 DPS310XTSA1, J1 ST-LINK Conn, J2 USB_C_2.0, J3 FFC2A32-24-T, J4 Screw_Terminal, J5 Screw_Terminal, J6 Screw_Terminal, J7 Screw_Terminal, Q1 MMBT3904-TP, Q2 MMBT3904-TP, Q3 FDN339AN, Q4 FDN339AN, Q5 SI7149ADP-T1-GE3, Q6 MMBT3904-TP, Q7 MMBT3904-TP, Q8 FDN339AN, Q9 FDN339AN, SW1 SW_SPDT, U1 STM32F103C8Tx, U10 TPS79133DBVR, U12 TLV709, U13 TLV75528PDBV, U2 AP63203WU, U3 ESP32-S3-WROOM-1, U4 TLV75515PDBV, U5 TLV709, U8 NEO-6M-GPS, U9 24AA32A-I_MS, Y1 16MHz

Commit message: fix
Parts:
- L2: footprint Inductor_SMD:L_0603_1608Metric -> Inductor_SMD:L_0402_1005Metric
- R44: footprint Resistor_SMD:R_0603_1608Metric -> Resistor_SMD:R_0402_1005Metric
Changed lines of the file:
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@@
 			)
 		)
-		(property "Footprint" "Resistor_SMD:R_0603_1608Metric"
+		(property "Footprint" "Resistor_SMD:R_0402_1005Metric"
 			(at 440.69 320.548 90)
 			(effects
@@
 			)
 		)
-		(property "Footprint" "Inductor_SMD:L_0603_1608Metric"
+		(property "Footprint" "Inductor_SMD:L_0402_1005Metric"
 			(at 450.85 318.77 0)
 			(effects
