File: KiCAD Files/Vertigo Daughterboard R1/_autosave-Vertigo Daughterboard R1.kicad_sch (KiCad schematic)
At the start: 21 parts, among them J1 Conn_01x08_Pin, U1 ICM-20602, U1 NEO-6M-GPS, U2 24AA32A-I_MS, U2 DPS310XTSA1

Commit message: PCB, Sensors, Pins etc
Parts:
- renumbered U1 to IC1, U2 to IC2
Changed lines of the file:
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@@
 		(dnp no)
 		(fields_autoplaced yes)
-		(property "Reference" "U2"
+		(property "Reference" "IC2"
 			(at 176.53 49.53 0)
 			(effects
@@
 			(project "Vertigo Daughterboard R1"
 				(path "/977084ba-e079-48e5-b203-f42a9d0a2d2c"
-					(reference "U2")
+					(reference "IC2")
 					(unit 1)
 				)
@@
 		(on_board yes)
 		(dnp no)
-		(property "Reference" "U1"
+		(property "Reference" "IC1"
 			(at 99.06 45.72 0)
 			(effects
@@
 			(project "Vertigo Daughterboard R1"
 				(path "/977084ba-e079-48e5-b203-f42a9d0a2d2c"
-					(reference "U1")
-					(unit 1)
-				)
+					(reference "IC1")
+					(unit 1)
+				)
